Commit message: Add files via upload

File: robots/pieter.urdf (robot description, URDF)
Before this commit: robot pieter, 5 links, 4 joints
Joints:
- joint front_axis: origin xyz=-0.462 0 0.0167 rpy=0 4.358E-17 1.5708 -> xyz=-0.462 0 0.0867 rpy=0 4.358E-17 1.5708
- joint left_axis: origin xyz=0.075 -0.232 0.0167 rpy=0 -7.4113E-17 0 -> xyz=0.075 -0.232 0.0867 rpy=0 -7.4113E-17 0
- joint rear_axis: origin xyz=0.6125 0 0.0167 rpy=0 4.358E-17 1.5708 -> xyz=0.6125 0 0.0867 rpy=0 4.358E-17 1.5708
- joint right_axis: origin xyz=0.075 0.225 0.0167 rpy=3.1415 6.123E-17 0 -> xyz=0.075 0.225 0.0867 rpy=3.1415 6.123E-17 0

Commit message: Add files via upload

File: robots/pieter.urdf (robot description, URDF)
Before this commit: robot pieter, 5 links, 4 joints
Joints:
- joint front_axis: origin xyz=-0.462 0 0.0167 rpy=0 4.358E-17 1.5708 -> xyz=-0.462 0 0.09 rpy=0 4.358E-17 1.5708; type continuous -> fixed
- joint left_axis: axis 1 0 0 -> 0 1 0; origin xyz=0.075 -0.232 0.0167 rpy=0 -7.4113E-17 0 -> xyz=0.075 -0.232 0.09 rpy=0 -7.4113E-17 0; type continuous -> fixed
- joint rear_axis: origin xyz=0.6125 0 0.0167 rpy=0 4.358E-17 1.5708 -> xyz=0.6125 0 0.09 rpy=0 4.358E-17 1.5708; type continuous -> fixed
- joint right_axis: axis -1 0 0 -> 0 -1 0; origin xyz=0.075 0.225 0.0167 rpy=3.1415 6.123E-17 0 -> xyz=0.075 0.225 0.09 rpy=3.1415 6.123E-17 0; type continuous -> fixed
